File: SparkFun_Buck-Boost.brd (EAGLE design)
At the start: 31.8 x 31.8 mm, 66 parts, among them U1 TPS63070

Commit message: V10 changes
- Added note for 2oz copper
- Replace power connections with 3.5mm screw terminals
Parts:
- removed J2: (no value), SparkFun-Connectors:1X02_NO_SILK
- added J4: (no value), SparkFun-Connectors:SCREWTERMINAL-3.5MM-2-NS
- added LOGO3: SPECIAL_INSTRUCTIONS-ORDERING, SparkFun-Aesthetics:ORDERING_INSTRUCTIONS
- J1: device SparkFun-Connectors:1X02_NO_SILK -> SparkFun-Connectors:SCREWTERMINAL-3.5MM-2-NS
- moved J1 27.7 mm to (29.0, 13.8)
- moved U$7 3.70 mm to (26.5, 11.0)
- moved U$5 3.54 mm to (0.51, 20.6)
- moved U$8 3.41 mm to (25.8, 20.2)
- moved U$6 3.18 mm to (0.51, 11.6)
- moved U$10 2.13 mm to (11.3, 17.8)
- moved U$13 2.05 mm to (28.3, 13.8)
- moved U$12 1.94 mm to (8.26, 14.2)
- moved U$14 1.91 mm to (28.3, 17.3)
- moved U$9 1.65 mm to (5.84, 8.26)
- moved LOGO2 1.61 mm to (27.8, 7.49)
- moved C5 0.64 mm to (21.5, 14.9)
- moved C7 0.64 mm to (21.5, 18.0)
- moved C1 0.63 mm to (10.3, 18.0)
- moved C2 0.63 mm to (10.3, 14.9)
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Connections:
- net GND: now also J4.2; no longer J2.1
- net VIN: now also J4.1; no longer J1.2
- net VOUT: now also J1.2; no longer J2.2
Routing:
- net VOUT: track 37.2 -> 38.5 mm
- net VIN: track 27.1 -> 26.5 mm
- net N$2: track 5.98 -> 6.49 mm
- net N$1: track 6.05 -> 6.56 mm
- net GND: vias 32 -> 34
Other:
- board text added: "- 2oz Copper!"

Commit message: Updated BOM
Replaced 357k resistor with 365k resistor
Parts:
- R4: value 357k -> 365k
Changed lines of the file:
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@@
 <attribute name="NAME" x="13.875" y="12.875" size="1.27" layer="25" rot="R90"/>
 <attribute name="PROD_ID" value="IC-14258" x="15.875" y="15.875" size="1.778" layer="27" rot="R90" display="off"/>
-<attribute name="VALUE" x="19.125" y="12.625" size="1.27" layer="27" rot="R90"/>
+<attribute name="VALUE" value="TPS63070" x="19.125" y="12.625" size="1.27" layer="27" rot="R90"/>
 </element>
 <element name="C1" library="SparkFun-Capacitors" package="0603" value="0.1uF" x="10.287" y="18.034" smashed="yes" rot="R90">
@@
 <attribute name="VALUE" x="16.891" y="10.16" size="0.6096" layer="27" font="vector" ratio="20" rot="R270" align="top-center"/>
 </element>
-<element name="R4" library="SparkFun-Resistors" package="0603" value="357k" x="16.129" y="10.16" smashed="yes" rot="R270">
+<element name="R4" library="SparkFun-Resistors" package="0603" value="365k" x="16.129" y="10.16" smashed="yes" rot="R270">
 <attribute name="NAME" x="16.891" y="10.16" size="0.6096" layer="25" font="vector" ratio="20" rot="R270" align="bottom-center"/>
 <attribute name="PROD_ID" value="RES-14262" x="16.129" y="10.16" size="1.778" layer="27" rot="R270" display="off"/>
-<attribute name="VALUE" x="15.367" y="10.16" size="0.6096" layer="27" font="vector" ratio="20" rot="R270" align="top-center"/>
+<attribute name="VALUE" value="365k" x="15.367" y="10.16" size="0.6096" layer="27" font="vector" ratio="20" rot="R270" align="top-center"/>
 </element>
 <element name="R5" library="SparkFun-Resistors" package="AXIAL-0.3" value="CUSTOM" x="9.525" y="8.382" smashed="yes" rot="R270">
